File: lv/kicad-template/template.kicad_sch (KiCad schematic)
At the start: 0 parts

Commit message: added aop amp system
Parts:
- added R1: R_Small, symbol Device:R_Small
- added R3: R_Small, Resistor_THT:R_Array_SIP7, symbol Device:R_Small
- added R5: 10k, symbol Device:R_Small
- added U7: LM393, symbol Comparator:LM393
Connections:
- new net: R1.2, R3.1, U7.3 (+)
- new net +5V: R1.1, R5.2
- new net GND: R3.2
- new net comp_out: R5.1, U7.1
- new net sensor_input: U7.2 (-)
- no-connect marks 0 -> 1
